File: Hand_motherboard/motherboard.brd (EAGLE design)
At the start: 44.1 x 39.4 mm, 22 parts, among them U1 ATXMEGA256A3-AU, U2 AZ1117EH, X1 52745-2090

Commit message: I think I figured out how gitignore works*
Parts:
- removed P4: (no value), jst-ph:JST-PH3
Connections:
- removed net ELECTRODE_D: P4.3, U1.9
- new net MOTOR_0D\: U1.17
- new net MOTOR_0U: U1.16
- new net MOTOR_1D: U1.19
- new net MOTOR_1U: U1.18
- new net MOTOR_2D: U1.21
- new net MOTOR_2U: U1.20
- new net MOTOR_3D: U1.23
- new net MOTOR_3U: U1.22
- new net SEL_0: U1.27
- new net SEL_1: U1.28
- new net SENSE_0: U1.8
- new net SENSE_1: U1.9
- new net SENSE_2: U1.10
- new net SENSE_3: U1.11
- net ANGLE: now also U1.13
- net ELECTRODE_A: now also U1.5; no longer U1.6
- net ELECTRODE_B: now also U1.4; no longer U1.7
- net ELECTRODE_C: now also U1.3; no longer U1.8
- net GND: no longer P4.2
- net MOTOR_11: no longer U1.36
- net MOTOR_12: no longer U1.37
- net MOTOR_21: no longer U1.38
- net MOTOR_22: no longer U1.39
- net MOTOR_31: no longer U1.40
- net MOTOR_32: no longer U1.41
- net MOTOR_41: no longer U1.42
- net MOTOR_42: no longer U1.43
- net MOTOR_EN: now also U1.26; no longer U1.31
- net PRESSURE: now also U1.12
- net SEL0: no longer U1.32
- net SEL1: no longer U1.33
- net VCC: no longer P4.1
Routing:
- net ELECTRODE_D: track 9.91 -> 0.00 mm
- net MOTOR_21: track 7.42 -> 0.02 mm
- net VCC: track 139.5 -> 134.2 mm
- net MOTOR_22: track 7.53 -> 4.05 mm
- net MOTOR_31: track 7.65 -> 4.19 mm
- net MOTOR_32: track 7.78 -> 4.37 mm
- net MOTOR_41: track 7.91 -> 4.53 mm
- net ELECTRODE_C: track 10.2 -> 7.51 mm
- net ELECTRODE_B: track 18.8 -> 16.8 mm
- net MOTOR_12: track 7.53 -> 6.12 mm
- net ELECTRODE_A: track 26.4 -> 25.2 mm
- net MOTOR_11: track 7.66 -> 6.42 mm
- net MOTOR_EN: track 17.8 -> 16.7 mm
- net SEL0: track 27.4 -> 26.5 mm
