File: Hand_motherboard/motherboard.sch (EAGLE design)
At the start: 22 parts, among them U1 ATXMEGA256A3-AU, U2 AZ1117EH, X1 52745-2090

Commit message: I think I figured out how gitignore works*
Parts:
- removed P4: (no value), jst-ph:JST-PH3
Connections:
- removed net ELECTRODE_D: P4.3, U1.PB3
- new net MOTOR_0D\: U1.PC1
- new net MOTOR_0U: U1.PC0
- new net MOTOR_1D: U1.PC3
- new net MOTOR_1U: U1.PC2
- new net MOTOR_2D: U1.PC5
- new net MOTOR_2U: U1.PC4
- new net MOTOR_3D: U1.PC7
- new net MOTOR_3U: U1.PC6
- new net SEL_0: U1.PD1
- new net SEL_1: U1.PD2
- new net SENSE_0: U1.PB2
- new net SENSE_1: U1.PB3
- new net SENSE_2: U1.PB4
- new net SENSE_3: U1.PB5
- net ANGLE: now also U1.PB7
- net ELECTRODE_A: now also U1.PA7; no longer U1.PB0
- net ELECTRODE_B: now also U1.PA6; no longer U1.PB1
- net ELECTRODE_C: now also U1.PA5; no longer U1.PB2
- net GND: no longer P4.2
- net MOTOR_11: no longer U1.PE0
- net MOTOR_12: no longer U1.PE1
- net MOTOR_21: no longer U1.PE2
- net MOTOR_22: no longer U1.PE3
- net MOTOR_31: no longer U1.PE4
- net MOTOR_32: no longer U1.PE5
- net MOTOR_41: no longer U1.PE6
- net MOTOR_42: no longer U1.PE7
- net MOTOR_EN: now also U1.PD0; no longer U1.PD5
- net PRESSURE: now also U1.PB6
- net SEL0: no longer U1.PD6
- net SEL1: no longer U1.PD7
- net VCC: no longer P4.1
